File: chassis_ctl_hardware/FDCAN_Transceiver.kicad_sch (KiCad schematic)
At the start: 3 parts, among them IC1 TJA1441AT

Commit message: Ver1.0
Parts:
- renumbered C10 to C18, C11 to C19
Changed lines of the file:
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@@
 		(in_pos_files yes)
 		(dnp no)
-		(property "Reference" "C10"
+		(property "Reference" "C18"
 			(at 113.792 76.454 0)
 			(show_name no)
@@
 			(project "chassis_ctl_hardware"
 				(path "/94505b12-11a5-48fa-b7fe-671b65f15652/d4fe4721-ecc1-4cb8-906b-7bb9251c3497"
-					(reference "C10")
+					(reference "C18")
 					(unit 1)
 				)
@@
 		(dnp no)
 		(fields_autoplaced yes)
-		(property "Reference" "#PWR024"
+		(property "Reference" "#PWR049"
 			(at 165.1 91.44 0)
 			(hide yes)
@@
 			(project "chassis_ctl_hardware"
 				(path "/94505b12-11a5-48fa-b7fe-671b65f15652/d4fe4721-ecc1-4cb8-906b-7bb9251c3497"
-					(reference "#PWR024")
+					(reference "#PWR049")
 					(unit 1)
 				)
@@
 		(in_pos_files yes)
 		(dnp no)
-		(property "Reference" "#PWR021"
+		(property "Reference" "#PWR047"
 			(at 116.84 54.61 0)
 			(hide yes)
@@
 			(project "chassis_ctl_hardware"
 				(path "/94505b12-11a5-48fa-b7fe-671b65f15652/d4fe4721-ecc1-4cb8-906b-7bb9251c3497"
-					(reference "#PWR021")
+					(reference "#PWR047")
 					(unit 1)
 				)
@@
 		(in_pos_files yes)
 		(dnp no)
-		(property "Reference" "#PWR0142"
+		(property "Reference" "#PWR048"
 			(at 152.4 60.96 0)
 			(hide yes)
@@
 			(project "chassis_ctl_hardware"
 				(path "/94505b12-11a5-48fa-b7fe-671b65f15652/d4fe4721-ecc1-4cb8-906b-7bb9251c3497"
-					(reference "#PWR0142")
+					(reference "#PWR048")
 					(unit 1)
 				)
@@
 		(in_pos_files yes)
 		(dnp no)
-		(property "Reference" "C11"
+		(property "Reference" "C19"
 			(at 148.082 76.454 0)
 			(show_name no)
@@
 			(project "chassis_ctl_hardware"
 				(path "/94505b12-11a5-48fa-b7fe-671b65f15652/d4fe4721-ecc1-4cb8-906b-7bb9251c3497"
-					(reference "C11")
-					(unit 1)
-				)
+					(reference "C19")
+					(unit 1)
+				)
