File: chassis_ctl_hardware/IMU.kicad_sch (KiCad schematic)
At the start: 4 parts, among them U1 ICM-40609-D

Commit message: Ver1.0
Parts:
- removed C1: 2.2μ, symbol Device:C
- added C7: 2.2μ, Capacitor_SMD:C_0603_1608Metric_Pad1.08x0.95mm_HandSolder, symbol Device:C
- C5: renamed from C2; footprint (none) -> Capacitor_SMD:C_0603_1608Metric_Pad1.08x0.95mm_HandSolder
- C6: renamed from C3; footprint (none) -> Capacitor_SMD:C_0603_1608Metric_Pad1.08x0.95mm_HandSolder
- renumbered U1 to U2
Connections:
- net CS is gone; now on net GND: U2.22 (NCS)
- net GND: now also C7.2
- net +5V renamed +3.3V
- net +3.3V: now also C7.1
Other:
- note added: "all capacitor ±10％"
