File: chassis_ctl_hardware/MCU_STM32_U545CET6.kicad_sch (KiCad schematic)
At the start: 15 parts, among them J7 STLink-v3mini, SW1 SW_Push, U3 STM32U545CET6, Y1 16M

Commit message: Second_Commit
Connections:
- net TIM1_CH1 is gone; now on net INT2/FSYNC: U3.29 (PA8)
- net TIM1_CH2 is gone; now on net INT1: U3.30 (PA9)
- net FDCAN_State: now also U3.20 (PB2); no longer U3.14 (PA4)
- net INT1: no longer U3.20 (PB2)
- net INT2/FSYNC: no longer U3.18 (PB0)
- net MCU_State_LED: now also U3.19 (PB1); no longer U3.13 (PA3)
- net SPI2_NSS: now reaches U3.25 (PB12)
- net I2C1_SCL: no longer names the net of U3.42 (PB6)
- net I2C1_SDA: no longer names the net of U3.43 (PB7)
- net SPI1_MISO renamed TIM3_CH1
- net SPI1_MOSI renamed TIM3_CH2
- net SPI1_SCK: no longer names the net of U3.15 (PA5)
- net TIM1_ETR renamed TIM2_CH3
- net TIM2_ETR: no longer names the net of U3.2 (PC13)
- new net TIM3_CH3: U3.18 (PB0)
- no-connect marks 15 -> 19
Changed lines of the file:
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@@
+	)
+	(no_connect
+		(at 44.45 102.87)
 	)
 	(no_connect
@@
 	)
 	(no_connect
-		(at 44.45 87.63)
-	)
-	(no_connect
 		(at 105.41 44.45)
 	)
@@
 	)
 	(no_connect
-		(at 44.45 113.03)
+		(at 105.41 41.91)
 	)
 	(no_connect
@@
 	)
 	(no_connect
+		(at 44.45 54.61)
+	)
+	(no_connect
+		(at 44.45 49.53)
+	)
+	(no_connect
+		(at 44.45 100.33)
+	)
+	(no_connect
 		(at 158.75 105.41)
 	)
@@
 	)
 	(no_connect
+		(at 44.45 52.07)
+	)
+	(no_connect
 		(at 146.05 105.41)
 	)
@@
 	(wire
 		(pts
-			(xy 119.38 52.07) (xy 105.41 52.07)
+			(xy 118.11 52.07) (xy 105.41 52.07)
 		)
 		(stroke
@@
 	(wire
 		(pts
-			(xy 44.45 92.71) (xy 22.86 92.71)
+			(xy 44.45 92.71) (xy 21.59 92.71)
 		)
 		(stroke
@@
 	)
 	(label "RCC_OSC_IN"
-		(at 119.38 52.07 180)
+		(at 118.11 52.07 180)
 		(effects
 			(font
@@
 	)
 	(label "JTDO_SWO"
-		(at 22.86 92.71 0)
+		(at 21.59 92.71 0)
 		(effects
 			(font
@@
 			)
 			(justify right bottom)
-		)
-	)
-	(hierarchical_label "FDCAN_State"
-		(shape output)
-		(at 44.45 52.07 180)
-		(effects
-			(font
-				(size 1.27 1.27)
-			)
-			(justify right)
 		)
 	)
@@
 		)
 	)
-	(hierarchical_label "TIM1_CH1"
+	(hierarchical_label "SPI2_NSS"
 		(shape input)
-		(at 44.45 62.23 180)
+		(at 44.45 113.03 180)
 		(effects
 			(font
@@
 		)
 	)
-	(hierarchical_label "TIM1_ETR"
+	(hierarchical_label "TIM2_CH3"
 		(shape input)
 		(at 44.45 46.99 180)
@@
 	(hierarchical_label "MCU_State_LED"
 		(shape output)
-		(at 44.45 49.53 180)
-		(effects
-			(font
-				(size 1.27 1.27)
-			)
-			(justify right)
-		)
-	)
-	(hierarchical_label "SPI1_MOSI"
+		(at 44.45 87.63 180)
+		(effects
+			(font
+				(size 1.27 1.27)
+			)
+			(justify right)
+		)
+	)
+	(hierarchical_label "FDCAN_State"
 		(shape output)
-		(at 44.45 59.69 180)
-		(effects
-			(font
-				(size 1.27 1.27)
-			)
-			(justify right)
-		)
-	)
-	(hierarchical_label "TIM1_CH2"
-		(shape input)
-		(at 44.45 64.77 180)
-		(effects
-			(font
-				(size 1.27 1.27)
-			)
-			(justify right)
-		)
-	)
-	(hierarchical_label "SPI1_MISO"
-		(shape input)
-		(at 44.45 57.15 180)
+		(at 44.45 90.17 180)
 		(effects
 			(font
@@
 		)
 	)
-	(hierarchical_label "I2C1_SCL"
+	(hierarchical_label "TIM3_CH3"
 		(shape input)
-		(at 44.45 100.33 180)
+		(at 44.45 85.09 180)
 		(effects
 			(font
@@
 		)
 	)
-	(hierarchical_label "TIM2_ETR"
-		(shape input)
-		(at 105.41 41.91 0)
-		(effects
-			(font
-				(size 1.27 1.27)
-			)
-			(justify left)
+	(hierarchical_label "INT1"
+		(shape output)
+		(at 44.45 64.77 180)
+		(effects
+			(font
+				(size 1.27 1.27)
+			)
+			(justify right)
 		)
 	)
@@
 		)
 	)
-	(hierarchical_label "INT2{slash}FSYNC"
-		(shape output)
-		(at 44.45 85.09 180)
-		(effects
-			(font
-				(size 1.27 1.27)
-			)
-			(justify right)
-		)
-	)
 	(hierarchical_label "TIM2_CH1"
 		(shape input)
@@
 		)
 	)
-	(hierarchical_label "SPI1_SCK"
+	(hierarchical_label "TIM3_CH1"
+		(shape input)
+		(at 44.45 57.15 180)
+		(effects
+			(font
+				(size 1.27 1.27)
+			)
+			(justify right)
+		)
+	)
+	(hierarchical_label "INT2{slash}FSYNC"
 		(shape output)
-		(at 44.45 54.61 180)
+		(at 44.45 62.23 180)
+		(effects
+			(font
+				(size 1.27 1.27)
+			)
+			(justify right)
+		)
+	)
+	(hierarchical_label "TIM3_CH2"
+		(shape input)
+		(at 44.45 59.69 180)
 		(effects
 			(font
@@
 		(effects
 			(font
-				(size 1.27 1.27)
-			)
-			(justify right)
-		)
-	)
-	(hierarchical_label "I2C1_SDA"
-		(shape input)
-		(at 44.45 102.87 180)
-		(effects
-			(font
-				(size 1.27 1.27)
-			)
-			(justify right)
-		)
-	)
-	(hierarchical_label "INT1"
-		(shape output)
-		(at 44.45 90.17 180)
-		(effects
-			(font
