File: chassis_ctl_hardware/chassis_ctl_hardware.kicad_sch (KiCad schematic)
At the start: 0 parts

Commit message: working
Parts:
- added J11: RJ45, Connector_RJ:RJ45_Amphenol_54602-x08_Horizontal, symbol Connector:RJ45
Connections:
- new net +5V: J11.4, J11.5
- new net CANH: J11.2, J11.6
- new net CANL: J11.1, J11.3
- new net GND: J11.7, J11.8
Other:
- added sheet FDCAN_Transceiver (FDCAN_Transceiver.kicad_sch)

Commit message: Ver1.0
Parts:
- added C1: 0.1u, Capacitor_SMD:C_0603_1608Metric_Pad1.08x0.95mm_HandSolder, symbol Device:C
- added C2: 0.47u, Capacitor_SMD:C_0603_1608Metric_Pad1.08x0.95mm_HandSolder, symbol Device:C
- added C3, C4: 1u, Capacitor_SMD:C_0603_1608Metric_Pad1.08x0.95mm_HandSolder, symbol Device:C
- added D1, D2: LED, LED_SMD:LED_0603_1608Metric_Pad1.05x0.95mm_HandSolder, symbol Device:LED
- added J1: USB_C, d_robo_lib:usb_c, symbol usb_can_hardware-rescue:USB_C_Receptacle_USB2.0-Connector
- added J2: Conn_01x05_Socket, Connector_JST:JST_XH_B5B-XH-A_1x05_P2.50mm_Vertical, symbol Connector:Conn_01x05_Socket
- added J3: encoder1, Connector_JST:JST_XH_S5B-XH-A_1x05_P2.50mm_Horizontal, symbol Connector:Conn_01x05_Socket
- added J4: encoder2, Connector_JST:JST_XH_S5B-XH-A_1x05_P2.50mm_Horizontal, symbol Connector:Conn_01x05_Socket
- added J5: Conn_01x04_Socket, Connector_JST:JST_XH_B4B-XH-A_1x04_P2.50mm_Vertical, symbol Connector:Conn_01x04_Socket
- added JP1: CC1, Jumper:SolderJumper-3_P1.3mm_Bridged12_RoundedPad1.0x1.5mm, symbol Jumper:SolderJumper_3_Bridged12
- added JP2: CC2, Jumper:SolderJumper-3_P1.3mm_Bridged12_RoundedPad1.0x1.5mm, symbol Jumper:SolderJumper_3_Bridged12
- added JP3: PWR, Jumper:SolderJumper-3_P1.3mm_Bridged12_RoundedPad1.0x1.5mm, symbol Jumper:SolderJumper_3_Bridged12
- added R1, R2: 4.7k, Resistor_SMD:R_0603_1608Metric_Pad0.98x0.95mm_HandSolder, symbol Device:R
- added R10, R11: 1k, Resistor_SMD:R_0603_1608Metric_Pad0.98x0.95mm_HandSolder, symbol Device:R
- added R3, R4, R5: 0, Resistor_SMD:R_0603_1608Metric_Pad0.98x0.95mm_HandSolder, symbol Device:R
- added R6, R7: 5.1k, Resistor_SMD:R_0603_1608Metric_Pad0.98x0.95mm_HandSolder, symbol Device:R
- added R8, R9: 56k, Resistor_SMD:R_0603_1608Metric_Pad0.98x0.95mm_HandSolder, symbol Device:R
- added U1: BU33SD5WG-TR, y-robo_footprint:SOT95P280X125-5N, symbol 2026-10-03_08-28-17:BU33SD5WG-TR
- renumbered J11 to J6
Connections:
- net +5V: now also C4.1, J3.2 (Pin_2), J4.2 (Pin_2), JP3.2 (C), U1.1 (VIN), U1.3 (STBY); no longer J6.4, J6.5
- net GND: now also C1.2, C2.2, C3.2, C4.2, J1.A1 (GND), J1.A12 (GND), J1.B1 (GND), J1.B12 (GND), J1.S1 (SHIELD), J2.5 (Pin_5), J3.5 (Pin_5), J4.5 (Pin_5), J5.4 (Pin_4), R6.1, R7.1, U1.2 (GND)
- new net: D1.2 (A), R10.2
- new net: JP2.1 (A), R7.2
- new net: JP2.3 (B), R9.1
- new net: J2.3 (Pin_3), R3.2
- new net: JP1.1 (A), R6.2
- new net: J2.2 (Pin_2), R4.2
- new net: JP1.3 (B), R8.1
- new net: J2.4 (Pin_4), R5.2
- new net: D2.2 (A), R11.2
- new net +3.3V: C3.1, J2.1 (Pin_1), J5.1 (Pin_1), R1.1, R10.1, R11.1, R2.1, U1.5 (VOUT)
- new net +5VA: J6.4, J6.5, JP3.1 (A)
- new net +5VD: C1.1, C2.1, J1.A4 (VBUS), J1.A9 (VBUS), J1.B4 (VBUS), J1.B9 (VBUS), JP3.3 (B), R8.2, R9.2
- new net CC1: J1.A5 (CC1), JP1.2 (C)
- new net CC2: J1.B5 (CC2), JP2.2 (C)
- new net D+: J1.A6 (D+), J1.B6 (D+)
- new net D-: J1.A7 (D-), J1.B7 (D-)
- new net I2C1_SCL: J5.2 (Pin_2), R1.2
- new net I2C1_SDA: J5.3 (Pin_3), R2.2
- new net MCU/FDCAN_State: D2.1 (K)
- new net MCU/MCU_State_LED: D1.1 (K)
- new net SPI2_MISO: R3.1
- new net SPI2_MOSI: R5.1
- new net SPI2_SCK: R4.1
- new net TIM1_CH1: J3.3 (Pin_3)
- new net TIM1_CH2: J3.1 (Pin_1)
- new net TIM1_ETR: J3.4 (Pin_4)
- new net TIM2_CH1: J4.3 (Pin_3)
- new net TIM2_CH2: J4.1 (Pin_1)
- new net TIM2_ETR: J4.4 (Pin_4)
- no-connect marks 0 -> 3
Other:
- added sheet MCU (MCU_STM32_U545CET6.kicad_sch)
- sheet IMU ports: added NSS; removed CS
- moved on the sheet: J6

Commit message: change PCB outline
Parts:
- added H1, H2, H3, H4: MountingHole, MountingHole:MountingHole_3.2mm_M3, symbol Mechanical:MountingHole
- J2: footprint Connector_JST:JST_XH_B5B-XH-A_1x05_P2.50mm_Vertical -> Connector_JST:JST_XH_S5B-XH-A_1x05_P2.50mm_Horizontal
- J5: footprint Connector_JST:JST_XH_B4B-XH-A_1x04_P2.50mm_Vertical -> Connector_JST:JST_XH_S4B-XH-A_1x04_P2.50mm_Horizontal
Connections:
- no-connect marks 3 -> 2

Commit message: Second_Commit
Parts:
- removed J2: Conn_01x05_Socket, Connector_JST:JST_XH_S5B-XH-A_1x05_P2.50mm_Horizontal, symbol Connector:Conn_01x05_Socket
- removed J5: Conn_01x04_Socket, Connector_JST:JST_XH_S4B-XH-A_1x04_P2.50mm_Horizontal, symbol Connector:Conn_01x04_Socket
- removed R1, R2: 4.7k, Resistor_SMD:R_0603_1608Metric_Pad0.98x0.95mm_HandSolder, symbol Device:R
- removed R3, R4, R5: 0, Resistor_SMD:R_0603_1608Metric_Pad0.98x0.95mm_HandSolder, symbol Device:R
Connections:
- net TIM1_CH1 is gone; now on net TIM2_CH1: J3.3 (Pin_3)
- net TIM1_CH2 is gone; now on net TIM2_CH2: J3.1 (Pin_1)
- net TIM2_CH1: no longer J4.3 (Pin_3)
- net TIM2_CH2: no longer J4.1 (Pin_1)
- net TIM1_ETR renamed TIM2_CH3
- net TIM2_ETR renamed TIM3_CH3
- new net TIM3_CH1: J4.3 (Pin_3)
- new net TIM3_CH2: J4.1 (Pin_1)
Other:
- sheet MCU ports: added SPI2_NSS, TIM2_CH3, TIM3_CH1, TIM3_CH2, TIM3_CH3; removed I2C1_SCL, I2C1_SDA, SPI1_MISO, SPI1_MOSI, SPI1_SCK, TIM1_CH1, TIM1_CH2, TIM1_ETR, TIM2_ETR
